Commit message: add eus model

File: jishupro/models/sample_model.urdf (robot description, URDF)
Before this commit: robot peco, 2 links, 1 joints
Links:
- removed link foot
- removed link leg
- added link lfoot, mass 1; visual mesh filename=file:///home/mech-user/jishupro_ws/src/CAD/model/link_foot.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
- added link lleg, mass 1; visual mesh filename=file:///home/mech-user/jishupro_ws/src/CAD/model/link_leg_l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
- added link lublock, mass 1; visual mesh filename=file:///home/mech-user/jishupro_ws/src/CAD/model/shoulder2.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
- added link rfoot, mass 1; visual mesh filename=file:///home/mech-user/jishupro_ws/src/CAD/model/link_foot.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
- added link rleg, mass 1; visual mesh filename=file:///home/mech-user/jishupro_ws/src/CAD/model/link_leg.S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
- added link root, mass 1; visual mesh filename=file:///home/mech-user/jishupro_ws/src/CAD/model/link_root.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
- added link rublock, mass 1; visual mesh filename=file:///home/mech-user/jishupro_ws/src/CAD/model/shoulder2.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
Joints:
- removed joint leg2foot
- added joint lleg2lfoot: type revolute, parent lleg, child lfoot, origin xyz=0.009 0 -0.210 rpy=0 0 0, axis 0 1 0, limit lower=-1.5 upper=1.5 effort=1000.0 velocity=0.5
- added joint lublock2lleg: type revolute, parent lublock, child lleg, origin xyz=0 0 -0.010 rpy=0 0 0, axis 0 1 0, limit lower=-1.5 upper=1.5 effort=1000.0 velocity=0.5
- added joint rleg2rfoot: type revolute, parent rleg, child rfoot, origin xyz=0.009 0 -0.210 rpy=0 0 0, axis 0 1 0, limit lower=-1.5 upper=1.5 effort=1000.0 velocity=0.5
- added joint root2lublock: type revolute, parent root, child lublock, origin xyz=0.2075 0.118 0.4054 rpy=0 0 0, axis 1 0 0, limit lower=-1.5 upper=1.5 effort=1000.0 velocity=0.5
- added joint root2rublock: type revolute, parent root, child rublock, origin xyz=0.2075 -0.118 0.4054 rpy=0 0 0, axis 1 0 0, limit lower=-1.5 upper=1.5 effort=1000.0 velocity=0.5
- added joint rublock2rleg: type revolute, parent rublock, child rleg, origin xyz=0 0 -0.010 rpy=0 0 0, axis 0 1 0, limit lower=-1.5 upper=1.5 effort=1000.0 velocity=0.5
