Commit message: aaa

File: jishupro/models/mbot.urdf (robot description, URDF)
Before this commit: robot mbot, 7 links, 6 joints
Joints:
- joint lleg2lfoot: limit lower=-1.5 upper=1.5 effort=1000.0 velocity=0.5 -> lower=-2.72 upper=1.5 effort=1000.0 velocity=0.5
- joint rleg2rfoot: limit lower=-1.5 upper=1.5 effort=1000.0 velocity=0.5 -> lower=-2.72 upper=1.5 effort=1000.0 velocity=0.5

Commit message: change initial value of wire length

File: jishupro/models/mbot.urdf (robot description, URDF)
Before this commit: robot mbot, 7 links, 6 joints
Joints:
- joint root2lublock: origin xyz=0.2075 0.118 0.4054 rpy=0 0 0 -> xyz=0.2075 0.118 0.4104 rpy=0 0 0
- joint root2rublock: origin xyz=0.2075 -0.118 0.4054 rpy=0 0 0 -> xyz=0.2075 -0.118 0.4104 rpy=0 0 0
